File: future-m2-goldfingers/module.kicad_pcb (KiCad board)
At the start: 4 copper layers, 22 x 42 mm, 44 parts, among them J1 M.2 Key M card edge (custom p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, J3 U.FL-R-SMT-1(01), U1 ESP32-C6FH8, U2 iCE40UP5K-SG48, U3 TLV75512PDBVR, Y1 40MHz / CL10pF

Commit message: Move the 3.3 V input bulk caps to the power contacts
C60, C61, C66 and C67 were meant to sit beside the power contacts but
were placed at the mounting end, 35 mm away, where they only dropped
into the planes through vias. They now sit at the contacts and feed
straight into the contacts' own In2 vias:

- C67 (22 uF) and C60 (10 uF) above contacts 70 and 72, each with a
  ground via;
- C61 (22 uF) and C66 (1 uF) in the strip east of the FPGA fan above
  contact 2, sharing one feed. The ESP bus lanes run under that strip,
  so their ground pads return through the front pour (recorded with the
  other pour-return deviations). The contact-1 ground via moves to
  (120.7, 137.75) to clear the feed.

Stitching vias that collided at the left end are dropped, and two
stitching vias keep the vacated NE corner tied to the planes.

ERC 0, DRC with parity 0, lint 24 infos (unchanged), quality errors
unchanged (31).

Co-Authored-By: Claude Opus 5.5 <noreply@anthropic.com>
Parts:
- moved C60 35.8 mm to (101.4, 135.0)
- moved C67 33.6 mm to (103.0, 135.0)
- moved C61 31.9 mm to (120.5, 135.9)
- moved C66 29.0 mm to (120.5, 132.8)
Routing:
- net +3.3V: track 42.8 -> 47.8 mm, vias 25 -> 21
- net GND: track 52.1 -> 50.4 mm, vias 59 -> 57

Commit message: Drop CRESET/CDONE straight into U2 and pull the ESP bus 1.7 mm west
CRESET and CDONE now turn west above the FPGA's east fan to vias on
the pin-8 / pin-7 via columns (115.25, 125.6) and (115.95, 126.3), so
their B.Cu hops are straight drops instead of diagonals across the
middle of the board. That frees x 116.4 .. 118.1 for the ESP bus: all
15 lanes move from 118.1 .. 121.6 to 116.4 .. 119.9, which shortens
every bus net by 1.2-1.4 mm on B.Cu (512.6 -> 491.2 mm in total for
the bus plus CRESET/CDONE).

With the lanes out of the strip above contact 2, C61 and C66 get their
ground vias back and drop off the pour-return deviation list.

ERC 0, DRC with parity 0, lint 24 infos (unchanged), quality errors
unchanged (31).

Co-Authored-By: Claude Opus 5.5 <noreply@anthropic.com>
Routing:
- net GND: track 50.4 -> 52.0 mm, vias 57 -> 59
- net ESP_GPIO23: track 42.1 -> 40.6 mm
- net ESP_GPIO16_TXD: track 32.6 -> 31.2 mm
- net USB_D+: track 30.7 -> 29.3 mm
- net ESP_GPIO5: track 33.1 -> 31.7 mm
- net ESP_GPIO22: track 40.9 -> 39.5 mm
- net ESP_GPIO21: track 39.8 -> 38.4 mm
- net ESP_GPIO19: track 34.5 -> 33.1 mm
- net ESP_EN: track 41.7 -> 40.3 mm
- net ESP_GPIO9_BOOT: track 31.8 -> 30.4 mm
- net ESP_GPIO4: track 33.6 -> 32.2 mm
- net ESP_GPIO20: track 36.8 -> 35.4 mm
- net USB_D-: track 30.8 -> 29.4 mm
- net ESP_GPIO8: track 32.4 -> 31.0 mm
- net ESP_GPIO17_RXD: track 33.2 -> 31.8 mm
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