File: future-m2-goldfingers/module.kicad_sch (KiCad schematic)
At the start: 44 parts, among them J1 M.2 Key M card edge (custom p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, J3 U.FL-R-SMT-1(01), U1 ESP32-C6FH8, U2 iCE40UP5K-SG48, U3 TLV75512PDBVR, Y1 40MHz / CL10pF

Commit message: Move the v2 module to the QFN40 ESP32-C6 with a 16 MB flash
U1 is now the flashless ESP32-C6 in QFN40 (LCSC C5364646, 0.4 mm pitch,
3.3 mm exposed pad; KiCad's QFN-40 land with the pad shrunk to match),
with a Winbond W25Q128JVPIQ 16 MB quad SPI flash (U4, LCSC C190862)
on SPI0/1 in QIO mode.

Pin changes: the QFN40 has GPIO10/11 but no GPIO14, so CRESET/CDONE
move to GPIO10/11 and GPIO18 is new on the connector (13 GPIOs + USB +
EN). The ESP bus grows to 16 back lanes; contact 33 (formerly ground)
carries GPIO4 through its old via, and the other ESP contacts shift one
slot east (USB is now on 26/24).

Layout: U1 moved 0.5 mm south to make room for the crystal's 0201 L5
and the 0201 VDDA1 cap. U4 sits in the north-east corner, rotated so
DI/CLK/HOLD fan straight into its south row; WP/DO/CS run up the east
side and WP/DO cross under CS on B.Cu above the chip (the flash pin
order is mirrored against the C6's). The flash runs from the 3.3 V
plane and VDD_SPI is left unconnected (it sits between the flash pins);
C68 0.1 uF decouples pin 8, C33 10 uF is 4 mm away. VDDPST2's plane and
ground vias sit on midlines between the B.Cu bus legs.

ERC 0, DRC with parity 0, lint 35 infos (no warnings), quality errors
31 (same accepted categories). New decoupling deviations recorded:
VDDPST1 2.7 mm, VDDPST2 2.4 mm, VDDA3P3 3.6 mm. L5 (24 nH 0201) still
needs an LCSC number.

Co-Authored-By: Claude Opus 5.5 <noreply@anthropic.com>
Parts:
- added C68: 0.1uF, Module2:C_0201, symbol Module2:C68
- added U4: W25Q128JVPIQ, Module2:WSON-8-1EP_6x5mm_P1.27mm_EP3.4x4.3mm, symbol Module2:U4
- C39: footprint Module2:C_0402 -> Module2:C_0201
- L5: footprint Module2:C_0402 -> Module2:L_0201
- U1: value ESP32-C6FH8 -> ESP32-C6; footprint Module2:QFN-32-1EP_5x5mm_P0.5mm_EP3.7x3.7mm -> Module2:QFN-40-1EP_5x5mm_P0.4mm_EP3.3x3.3mm
Connections:
- net +3.3V: now also U1.28 (VDDPST2), U1.37 (VDDA1), U1.40 (VDDA2), C68.1, U4.8 (VCC); no longer U1.20 (VDDPST2), U1.29 (VDDA1), U1.32 (VDDA2)
- net ESP_GPIO15: now also J1.22, U1.27 (GPIO15); no longer J1.20, U1.19 (GPIO15)
- net ESP_GPIO16_TXD: now also J1.20, U1.29 (GPIO16/U0TXD); no longer J1.18, U1.21 (GPIO16/U0TXD)
- net ESP_GPIO17_RXD: now also J1.18, U1.30 (GPIO17/U0RXD); no longer J1.16, U1.22 (GPIO17/U0RXD)
- net ESP_GPIO19: now also U1.32 (GPIO19); no longer U1.24 (GPIO19)
- net ESP_GPIO20: now also U1.33 (GPIO20); no longer U1.25 (GPIO20)
- net ESP_GPIO21: now also U1.34 (GPIO21); no longer U1.26 (GPIO21)
- net ESP_GPIO22: now also U1.35 (GPIO22); no longer U1.27 (GPIO22)
- net ESP_GPIO23: now also U1.36 (GPIO23); no longer U1.28 (GPIO23)
- net ESP_GPIO4: now also J1.33; no longer J1.32
- net ESP_GPIO5: now also J1.32; no longer J1.30
- net ESP_GPIO8: now also J1.30; no longer J1.28
- net ESP_GPIO9_BOOT: now also J1.28; no longer J1.26
- net FPGA_CDONE: now also U1.17 (GPIO11); no longer U1.23 (GPIO18)
- net FPGA_CRESET_N: now also U1.16 (GPIO10); no longer U1.18 (GPIO14)
- net GND: now also U1.41 (GND), C68.2, U4.4 (GND), U4.9 (EP); no longer J1.33, U1.33 (GND)
- net USB_D+: now also J1.24, U1.19 (GPIO13/USB_D+); no longer J1.22, U1.17 (GPIO13/USB_D+)
- net USB_D-: now also J1.26, U1.18 (GPIO12/USB_D-); no longer J1.24, U1.16 (GPIO12/USB_D-)
- net XTAL_N: now also U1.38 (XTAL_N); no longer U1.30 (XTAL_N)
- net XTAL_P: now also U1.39 (XTAL_P); no longer U1.31 (XTAL_P)
- new net ESP_GPIO18: J1.16, U1.31 (GPIO18)
- new net FLASH_CLK: U1.25 (SPICLK), U4.6 (CLK)
- new net FLASH_CS: U1.20 (SPICS0), U4.1 (/CS)
- new net FLASH_DI: U1.26 (SPID), U4.5 (DI(IO0))
- new net FLASH_DO: U1.21 (SPIQ), U4.2 (DO(IO1))
- new net FLASH_HD: U1.24 (SPIHD), U4.7 (/HOLD(IO3))
- new net FLASH_WP: U1.22 (SPIWP), U4.3 (/WP(IO2))
- no-connect marks 1 -> 2
Other:
- note added: "+3.3V: ESP VDDPST1/2, VDDA1/2; flash VCC; FPGA VCCIO/VPP; input bulk at the card edge"
- note added: "ESP32-C6 (QFN40, external flash U4; VDD_SPI unused)"
- note added: "PWR_FLAGs: +3.3V and GND enter on card-edge contacts 2/4/70/72/74 and 1/3/9/15/21/27/39/45/51/57/71/73/75."
- note added: "W25Q128JV 16 MB quad SPI flash (3.3 V from the plane)"
- note removed: "+3.3V: ESP VDDPST1/2, VDDA1/2; FPGA VCCIO/VPP; input bulk at the card edge"
- note removed: "ESP32-C6FH8 (QFN32, 8 MB in-package flash)"
- note removed: "PWR_FLAGs: +3.3V and GND enter on card-edge contacts 2/4/70/72/74 and 1/3/9/15/21/27/33/39/45/51/57/71/73/75."
- moved on the sheet: C46, C48, C49, C50, C52, C60, C61, C66, C67
